File: daq_overview.kicad_sch (KiCad schematic)
At the start: 15 parts

Commit message: Add Califa and most of bus daq. Started data stream overview.
Parts:
- added CLK_TRG_DISTR2, CLK_TRG_DISTR3, CLK_TRG_DISTR4, CLK_TRG_DISTR5, CLK_TRG_DISTR6: ~, symbol daq_parts:clk_trg_distr2
- added CLK_TRG_DISTR7, CLK_TRG_DISTR8: ~, symbol daq_parts:clk_trg_distr1
- added EXPLODER2, EXPLODER3, EXPLODER4: ~, symbol daq_parts:exploder3
- added FEBEX_CONTROLLER1, FEBEX_CONTROLLER2, FEBEX_CONTROLLER3, FEBEX_CONTROLLER4: ~, symbol daq_parts:febex_controller
- added KINPEX1: ~, symbol daq_parts:kinpex
- added LXIR133:7720: ~, symbol daq_parts:daq_pc
- added NIM_CFD1: ~, symbol daq_parts:nim_cfd
- added NIM_FIFO1: ~, symbol daq_parts:nim_fifo
- added PEXARIA2: ~, symbol daq_parts:pexaria5
- added R4L-56, X86L-134, X86L-135, X86L-162, X86L-163, X86L-91: ~, symbol daq_parts:daq_node_source
- added TRIXOR10, TRIXOR2, TRIXOR3, TRIXOR4, TRIXOR5, TRIXOR6, TRIXOR7, TRIXOR8, TRIXOR9: ~, symbol daq_parts:trixor
Connections:
- net DEADTIME: now also EXPLODER2. (USB), TRIXOR2. (TRIGGER_BUS_B)
- net TRIGGER: now also EXPLODER2. (USB), PEXARIA2. (WHITE_RABBIT_IN)
- net TRIGGER_BUS_BUSDAQ: now also TRIXOR10. (TRIGGER_BUS_B), TRIXOR2. (TRIGGER_BUS_B), TRIXOR3. (TRIGGER_BUS_B), TRIXOR4. (TRIGGER_BUS_B), TRIXOR5. (TRIGGER_BUS_B), TRIXOR6. (TRIGGER_BUS_B), TRIXOR7. (TRIGGER_BUS_B)
- net TRIGGER_NEULAND: now also NIM_FIFO1. (OUT4)
- net WHITE_RABBIT_TS: now also PEXARIA2. (WHITE_RABBIT_IN)
- net at DIGILENT_HS1. (USB): now also RASPBERRY_PI1. (USB_POWER); no longer WRTCLK1. (USB)
- new net: LXIR133:7720. (ETH_OUT), R4L-56. (ETH_OUT), X86L-134. (ETH_OUT), X86L-135. (ETH_OUT), X86L-162. (ETH_OUT), X86L-163. (ETH_OUT), X86L-91. (ETH_OUT)
- new net: TRIXOR5. (TRIGGER_BUS_B), TRIXOR6. (TRIGGER_BUS_B)
- new net: CLK_TRG_DISTR6. (TRIGGER_OUT2), CLK_TRG_DISTR8. (TRIGGER_IN)
- new net: CLK_TRG_DISTR6. (TRIGGER_OUT2), CLK_TRG_DISTR7. (TRIGGER_IN)
- new net: TRIXOR3. (TRIGGER_BUS_B), TRIXOR4. (TRIGGER_BUS_B)
- new net: DIGILENT_HS1. (USB), WRTCLK1. (USB)
- new net: EXPLODER3. (USB), FEBEX_CONTROLLER2. (TRIGGER_BUS), FEBEX_CONTROLLER4. (TRIGGER_BUS)
- new net: FEBEX_CONTROLLER4. (TRIGGER_BUS), KINPEX1. (SFP_FIBER1)
- new net: TRIVA2. (TRIGGER_BUS_B), VULOM2. (LEMO_OUT2)
- new net: CLK_TRG_DISTR1. (TRIGGER_OUT2), VFTX1. (SMA_IN9)
- new net: PEXARIA1. (WHITE_RABBIT_IN), WRTCLK_HDMI_ADAPTER1. (LVDS_OUT8)
- new net: FEBEX_CONTROLLER2. (TRIGGER_BUS), KINPEX1. (SFP_FIBER1)
- new net: FEBEX_CONTROLLER3. (TRIGGER_BUS), KINPEX1. (SFP_FIBER1)
- new net: FEBEX_CONTROLLER1. (TRIGGER_BUS), KINPEX1. (SFP_FIBER1)
- new net: TRIXOR7. (TRIGGER_BUS_B), TRIXOR8. (TRIGGER_BUS_B)
- new net: EXPLODER2. (USB), FEBEX_CONTROLLER1. (TRIGGER_BUS), FEBEX_CONTROLLER3. (TRIGGER_BUS)
- new net: NIM_CFD1. (OUT3), NIM_FIFO1. (OUT4)
- new net: TRIXOR8. (TRIGGER_BUS_B), TRIXOR9. (TRIGGER_BUS_B)
- new net: CLK_TRG_DISTR2. (TRIGGER_OUT2), CLK_TRG_DISTR3. (TRIGGER_OUT2)
- new net: EXPLODER2. (USB), EXPLODER4. (USB)
- new net: TRIXOR10. (TRIGGER_BUS_B), TRIXOR9. (TRIGGER_BUS_B)
- new net: CLK_TRG_DISTR2. (TRIGGER_OUT2), CLK_TRG_DISTR4. (TRIGGER_OUT2)
- new net: EXPLODER2. (USB), EXPLODER3. (USB)
- new net CLK_TRG_FOR_FIBER: CLK_TRG_DISTR2. (TRIGGER_OUT2)
- new net CLK_TRG_FOR_NEULAND: CLK_TRG_DISTR6. (TRIGGER_OUT2)
- new net CLK_TRG_FOR_TOFD: CLK_TRG_DISTR5. (TRIGGER_OUT2)
- new net ENCODED_TRIG: EXPLODER2. (USB), TRIXOR2. (TRIGGER_BUS_B)
- new net NEULAND_MULTIPLICITY: NIM_CFD1. (OUT3)
- no-connect marks 4 -> 7
Other:
- note added: "CALIFA"
- note added: "DATA STREAM OVERVIEW"
- note added: "FIBER"
- note added: "LOS"
- note added: "MAIN FIBER CLOCK_DISTR"
- note added: "MASTER"
- note added: "NEULAND"
- note added: "NOTE: Connections not verified! And not complete!"
- note added: "OVERLORD EXPLODER"
- note added: "Required signals: - WHITE_RABBIT_TS connected to upstream White Rabbit switch"
- note added: "SLAVE"
- note added: "TOFD"
- note added: "Where does this come from?"
- note added: "X86L-101 (NLR0)"
- note added: "X86L-102 (NLR1)"
- note added: "X86L-134 (FIBER3032)"
- note added: "X86L-135 (FIBER3133)"
- note added: "X86L-162 (TOFD34)"
- note added: "X86L-163 (TOFD12)"
- note added: "X86L-75 (mes0)"
- note added: "X86L-77 (NLL1)"
- note added: "X86L-80 (NLL0)"
- note added: "X86L-91 (LOS TAMEX)"
- note removed: "X86L-91"
- moved on the sheet: TRIXOR1

Commit message: Add things in data flow.
Parts:
- added DE10NANO1, DE10NANO11, DE10NANO12, DE10NANO13, DE10NANO2, DE10NANO4, DE10NANO6, DE10NANO7, MOSAIC1, R4L-44_TTT10, R4L-57_MAIN, R4L-71_MUSIC, X86L-101_NLR0, X86L-102_NLR1, X86L-77_NLL1, X86L-80_NLL0: ~, symbol daq_parts:daq_node_source
- added FOOT_TIME_STITCHER, TIME_STITCHER: ~, symbol daq_parts:ucesb
- added LANDGW01:9000_FOOT_TIMESORTER, LXLANDDAQ01_TIME_SORTER: ~, symbol daq_parts:time_sorter
- added LANDGW01_RPC_FILTER, LXIR133:7700, LXIR133:7760, LXIR133:7800, SFSPC005_ALPIDE1: ~, symbol daq_parts:daq_node_merger
- added TRB3_MBS_NODE, X86L-108_CALIFA_WIX1, X86L-109_CALIFA_MES1, X86L-75_CALIFA_MES0, X86L-76_CALIFA_WIX0: ~, symbol daq_parts:daq_node_source_mbs
- LXIR133:7720: symbol daq_parts:daq_pc -> daq_parts:daq_node_merger
- renumbered R4L-56 to R4L-56_LOS_VFTX, X86L-134 to X86L-134_FIB3032, X86L-135 to X86L-135_FIB3133, X86L-162 to X86L-162_TOFD34, X86L-163 to X86L-163_TOFD12, X86L-91 to X86L-91_LOS_TAMEX
Connections:
- net at LXIR133:7720. (DRASI_OUT), R4L-56_LOS_VFTX. (DRASI_OUT), X86L-134_FIB3032. (DRASI_OUT)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: now also X86L-101_NLR0. (DRASI_OUT), X86L-102_NLR1. (DRASI_OUT), X86L-77_NLL1. (DRASI_OUT), X86L-80_NLL0. (DRASI_OUT)
- net at CLK_TRG_DISTR8. (TRIGGER_IN): no longer CLK_TRG_DISTR6. (TRIGGER_OUT2)
- net at CLK_TRG_DISTR7. (TRIGGER_IN): no longer CLK_TRG_DISTR6. (TRIGGER_OUT2)
- net at DIGILENT_HS1. (USB): now also RASPBERRY_PI1. (USB_POWER); no longer WRTCLK1. (USB)
- net at KINPEX1. (SFP_FIBER1): now also FEBEX_CONTROLLER1. (TRIGGER_BUS); no longer FEBEX_CONTROLLER3. (TRIGGER_BUS)
- net at FEBEX_CONTROLLER1. (TRIGGER_BUS): now also EXPLODER2. (USB), FEBEX_CONTROLLER3. (TRIGGER_BUS); no longer KINPEX1. (SFP_FIBER1)
- net at TRIXOR8. (TRIGGER_BUS_B): now also TRIXOR9. (TRIGGER_BUS_B); no longer TRIXOR7. (TRIGGER_BUS_B)
- net at TRIXOR9. (TRIGGER_BUS_B): no longer TRIXOR8. (TRIGGER_BUS_B)
- net at CLK_TRG_DISTR3. (TRIGGER_OUT2): now also CLK_TRG_DISTR2. (TRIGGER_OUT2)
- net at LXIR133:7720. (DRASI_OUT): now also LANDGW01:9000_FOOT_TIMESORTER. (TRANSPORT), LANDGW01_RPC_FILTER. (DRASI_OUT), LXIR133:7700. (DRASI_OUT), LXIR133:7760. (DRASI_OUT), LXIR133:7800. (DRASI_OUT), LXLANDDAQ01_TIME_SORTER. (TRANSPORT), SFSPC005_ALPIDE1. (DRASI_OUT)
- net at EXPLODER4. (USB): now also EXPLODER2. (USB)
- net at CLK_TRG_DISTR4. (TRIGGER_OUT2): now also CLK_TRG_DISTR2. (TRIGGER_OUT2)
- net at EXPLODER3. (USB): no longer EXPLODER2. (USB)
- new net: TRIXOR5. (TRIGGER_BUS_B), TRIXOR6. (TRIGGER_BUS_B)
- new net: CLK_TRG_DISTR6. (TRIGGER_OUT2), CLK_TRG_DISTR8. (TRIGGER_IN)
- new net: CLK_TRG_DISTR6. (TRIGGER_OUT2), CLK_TRG_DISTR7. (TRIGGER_IN)
- new net: DE10NANO1. (DRASI_OUT), DE10NANO11. (DRASI_OUT), DE10NANO12. (DRASI_OUT), DE10NANO13. (DRASI_OUT), DE10NANO2. (DRASI_OUT), DE10NANO4. (DRASI_OUT), DE10NANO6. (DRASI_OUT), DE10NANO7. (DRASI_OUT), LANDGW01:9000_FOOT_TIMESORTER. (TRANSPORT)
- new net: TRIXOR3. (TRIGGER_BUS_B), TRIXOR4. (TRIGGER_BUS_B)
- new net: DIGILENT_HS1. (USB), WRTCLK1. (USB)
- new net: LXIR133:7760. (DRASI_OUT), R4L-44_TTT10. (DRASI_OUT)
- new net: FOOT_TIME_STITCHER. (TRANSPORT), LANDGW01:9000_FOOT_TIMESORTER. (TRANSPORT)
- new net: LXIR133:7700. (DRASI_OUT), R4L-57_MAIN. (DRASI_OUT)
- new net: EXPLODER3. (USB), FEBEX_CONTROLLER2. (TRIGGER_BUS), FEBEX_CONTROLLER4. (TRIGGER_BUS)
- new net: TRIVA2. (TRIGGER_BUS_B), VULOM2. (LEMO_OUT2)
- new net: CLK_TRG_DISTR1. (TRIGGER_OUT2), VFTX1. (SMA_IN9)
- new net: PEXARIA1. (WHITE_RABBIT_IN), WRTCLK_HDMI_ADAPTER1. (LVDS_OUT8)
- new net: MOSAIC1. (DRASI_OUT), SFSPC005_ALPIDE1. (DRASI_OUT)
- new net: FEBEX_CONTROLLER3. (TRIGGER_BUS), KINPEX1. (SFP_FIBER1)
- new net: LXLANDDAQ01_TIME_SORTER. (TRANSPORT), TIME_STITCHER. (TRANSPORT)
- new net: TRIXOR7. (TRIGGER_BUS_B), TRIXOR8. (TRIGGER_BUS_B)
- new net: LXLANDDAQ01_TIME_SORTER. (TRANSPORT), X86L-108_CALIFA_WIX1. (TRANSPORT), X86L-109_CALIFA_MES1. (TRANSPORT), X86L-75_CALIFA_MES0. (TRANSPORT), X86L-76_CALIFA_WIX0. (TRANSPORT)
- new net: LXIR133:7800. (DRASI_OUT), R4L-71_MUSIC. (DRASI_OUT)
- new net: NIM_CFD1. (OUT3), NIM_FIFO1. (OUT4)
- new net: TRIXOR10. (TRIGGER_BUS_B), TRIXOR9. (TRIGGER_BUS_B)
- new net: EXPLODER2. (USB), EXPLODER3. (USB)
- new net TRANSPORT: LANDGW01_RPC_FILTER. (DRASI_OUT), TRB3_MBS_NODE. (TRANSPORT)
- now unconnected: EXPLODER3. (USB), TRIXOR9. (TRIGGER_BUS_B)
Other:
- note added: "BUS"
- note added: "Event builder data output ports: * transport: 7xx1 * stream: 7xx2 * server: 7xx3 <-(connect here) config: lxir133:7xx0/eb.bash"
- note added: "FOOT"
- note added: "FOOT time sorter data output ports: * drasi: 9000 * stream: 8001, 8002 config: krpc003:r3bfoot/to/to.bash"
- note added: "RPC config: * drasi filter: ~/http/drasi/f_user_example/filter_trbts2lmdwr.c * start script: ~/htt/rpc/wr_reorder.sh * stream port: MBS default"
- note added: "Time sorter data output ports: * transport: MBS default * stream: MBS default * server: 9100 <-(connect here) config: lxlanddaq01/to.bash"
- note added: "Time stitcher data output ports: * stream: 8003 <-(connect here) config: krpc003:r3bfoot/st/st.bash"
- note added: "Time stitcher data output ports: * transport: 8000 * stream: 9000 <-(online connect here) config: scripts/timestitcher.sh"
- moved on the sheet: LXIR133:7720

Commit message: Add comment for repo address and big title.
Parts:
- renumbered TRB3_MBS_NODE to TRB3_MBS_NODE:DAQ-RPC-R3B
Connections:
- net at CLK_TRG_DISTR8. (TRIGGER_IN): no longer CLK_TRG_DISTR6. (TRIGGER_OUT2)
- net at CLK_TRG_DISTR7. (TRIGGER_IN): no longer CLK_TRG_DISTR6. (TRIGGER_OUT2)
- net at DIGILENT_HS1. (USB): now also RASPBERRY_PI1. (USB_POWER); no longer WRTCLK1. (USB)
- net at LANDGW01:9000_FOOT_TIMESORTER. (TRANSPORT): now also FOOT_TIME_STITCHER. (TRANSPORT)
- net at FOOT_TIME_STITCHER. (TRANSPORT): no longer LANDGW01:9000_FOOT_TIMESORTER. (TRANSPORT)
- net at KINPEX1. (SFP_FIBER1): now also FEBEX_CONTROLLER1. (TRIGGER_BUS); no longer FEBEX_CONTROLLER3. (TRIGGER_BUS)
- net at FEBEX_CONTROLLER1. (TRIGGER_BUS): now also EXPLODER2. (USB), FEBEX_CONTROLLER3. (TRIGGER_BUS); no longer KINPEX1. (SFP_FIBER1)
- net at TIME_STITCHER. (TRANSPORT): now also LXLANDDAQ01_TIME_SORTER. (TRANSPORT)
- net at LXLANDDAQ01_TIME_SORTER. (TRANSPORT): now also X86L-108_CALIFA_WIX1. (TRANSPORT), X86L-109_CALIFA_MES1. (TRANSPORT), X86L-75_CALIFA_MES0. (TRANSPORT), X86L-76_CALIFA_WIX0. (TRANSPORT); no longer TIME_STITCHER. (TRANSPORT)
- net at TRIXOR8. (TRIGGER_BUS_B): now also TRIXOR9. (TRIGGER_BUS_B); no longer TRIXOR7. (TRIGGER_BUS_B)
- net at TRIXOR9. (TRIGGER_BUS_B): no longer TRIXOR8. (TRIGGER_BUS_B)
- net at CLK_TRG_DISTR3. (TRIGGER_OUT2): now also CLK_TRG_DISTR2. (TRIGGER_OUT2)
- net at EXPLODER4. (USB): now also EXPLODER2. (USB)
- net at CLK_TRG_DISTR4. (TRIGGER_OUT2): now also CLK_TRG_DISTR2. (TRIGGER_OUT2)
- net at EXPLODER3. (USB): no longer EXPLODER2. (USB)
- new net: TRIXOR5. (TRIGGER_BUS_B), TRIXOR6. (TRIGGER_BUS_B)
- new net: CLK_TRG_DISTR6. (TRIGGER_OUT2), CLK_TRG_DISTR8. (TRIGGER_IN)
- new net: CLK_TRG_DISTR6. (TRIGGER_OUT2), CLK_TRG_DISTR7. (TRIGGER_IN)
- new net: TRIXOR3. (TRIGGER_BUS_B), TRIXOR4. (TRIGGER_BUS_B)
- new net: DIGILENT_HS1. (USB), WRTCLK1. (USB)
- new net: LANDGW01:9000_FOOT_TIMESORTER. (TRANSPORT), LANDGW01_RPC_FILTER. (DRASI_OUT), LXIR133:7700. (DRASI_OUT), LXIR133:7720. (DRASI_OUT), LXIR133:7760. (DRASI_OUT), LXIR133:7800. (DRASI_OUT), LXLANDDAQ01_TIME_SORTER. (TRANSPORT), SFSPC005_ALPIDE1. (DRASI_OUT)
- new net: EXPLODER3. (USB), FEBEX_CONTROLLER2. (TRIGGER_BUS), FEBEX_CONTROLLER4. (TRIGGER_BUS)
- new net: TRIVA2. (TRIGGER_BUS_B), VULOM2. (LEMO_OUT2)
- new net: CLK_TRG_DISTR1. (TRIGGER_OUT2), VFTX1. (SMA_IN9)
- new net: PEXARIA1. (WHITE_RABBIT_IN), WRTCLK_HDMI_ADAPTER1. (LVDS_OUT8)
- new net: FEBEX_CONTROLLER3. (TRIGGER_BUS), KINPEX1. (SFP_FIBER1)
- new net: TRIXOR7. (TRIGGER_BUS_B), TRIXOR8. (TRIGGER_BUS_B)
- new net: NIM_CFD1. (OUT3), NIM_FIFO1. (OUT4)
- new net: TRIXOR10. (TRIGGER_BUS_B), TRIXOR9. (TRIGGER_BUS_B)
- new net: EXPLODER2. (USB), EXPLODER3. (USB)
- now unconnected: EXPLODER3. (USB), TRIXOR9. (TRIGGER_BUS_B), X86L-108_CALIFA_WIX1. (TRANSPORT), X86L-109_CALIFA_MES1. (TRANSPORT), X86L-75_CALIFA_MES0. (TRANSPORT), X86L-76_CALIFA_WIX0. (TRANSPORT)
Other:
- note added: "DAQ 202402_s118"
Changed lines of the file:
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@@
 (kicad_sch (version 20230121) (generator eeschema)
   (paper "A0")
+  (title_block
+    (date "2023-11-28")
+    (comment 1 "repository: git@github.com:bl0x/daq_overview.git")
+  )
   (junction (at 750.57 800.1) (diameter 0) (color 0 0 0 0)
   )
@@
     (effects (font (size 5 5)) (justify left bottom))
   )
+  (text "DAQ 202402_s118" (at 889 49.53 0)
+    (effects (font (size 20 20) bold) (justify left bottom))
+  )
   (text "X86L-163 (TOFD12)\n" (at 674.37 250.19 0)
     (effects (font (size 3 3)) (justify left bottom))
@@
   (symbol (lib_id "daq_parts:daq_node_source_mbs") (at 784.86 664.21 0) (unit 1)
     (in_bom yes) (on_board yes) (dnp no)
-    (property "Reference" "TRB3_MBS_NODE" (at 784.86 647.7 0)
+    (property "Reference" "TRB3_MBS_NODE:DAQ-RPC-R3B" (at 784.86 647.7 0)
       (effects (font (size 1.27 1.27)))
     )
@@
       (project "daq_overview"
         (path "/e1579a50-ec5d-40e2-abf2-cd20f2752378"
-          (reference "TRB3_MBS_NODE") (unit 1)
+          (reference "TRB3_MBS_NODE:DAQ-RPC-R3B") (unit 1)
         )
       )
